File: kicad/Meteostation_3/Meteostation.sch (KiCad schematic (older format))
At the start: 94 parts, among them J1 TxD, J12 TxD_AirS8, J13 RxD_AirS8, J14 +5v, J2 RxD, J3 BME280_SCL, J4 BME280_SDA, J5 RST, J6 +EXT, J7 -EXT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

Commit message: изменено:      kicad/Meteostation_3/Meteostation.kicad_pcb 	изменено:      kicad/Meteostation_3/Meteostation.kicad_pcb-bak 	изменено:      kicad/Meteostation_3/Meteostation.sch 	изменено:      kicad/Meteostation_3/Meteostation.sch-bak 	изменено:      kicad/Meteostation_3/gerber/Border.gbr 	изменено:      kicad/Meteostation_3/gerber/Bottom.gbr 	изменено:      kicad/Meteostation_3/gerber/MaskBottom.gbr 	изменено:      kicad/Meteostation_3/gerber/MaskTop.gbr 	изменено:      kicad/Meteostation_3/gerber/Meteostation-job.gbrjob 	изменено:      kicad/Meteostation_3/gerber/Meteostation.zip 	изменено:      kicad/Meteostation_3/gerber/NCData.drl 	изменено:      kicad/Meteostation_3/gerber/Top.gbr
Connections:
- net +3.3VDAC: now also D3.43 (PMODE2), D3.44 (PMODE1)
- net GND: no longer D3.43 (PMODE2), D3.44 (PMODE1)
Changed lines of the file:
@@
 	7650 8550 8700 8550
-$Comp
-L power:GND #PWR0106
-U 1 1 630D5B6C
-P 6150 6850
-F 0 "#PWR0106" H 6150 6600 50  0001 C CNN
-F 1 "GND" H 6155 6677 50  0001 C CNN
-F 2 "" H 6150 6850 50  0001 C CNN
-F 3 "" H 6150 6850 50  0001 C CNN
-	1    6150 6850
-	-1   0    0    1
-$EndComp
-Wire Wire Line
-	6150 6850 6150 6950
-Connection ~ 6150 6950
 $Comp
 L Meteostation-rescue:MC33375ST-My_Library D1
@@
 	9650 3500 9650 3650
 Connection ~ 9650 3500
+Wire Wire Line
+	6150 6950 6250 6950
+Connection ~ 6150 6950
+Connection ~ 6250 6950
 $EndSCHEMATC

Commit message: изменено:      kicad/BME280/fp-info-cache 	изменено:      kicad/Meteostation_3/Meteostation.sch 	изменено:      kicad/Meteostation_3/Meteostation.sch-bak
Parts:
- D13, D8: value MBR0540 -> F7
Changed lines of the file:
@@
 P 7900 5500
 F 0 "D8" H 7900 5350 50  0000 C CNN
-F 1 "MBR0540" H 7800 5350 50  0001 C CNN
+F 1 "F7" H 7800 5350 50  0001 C CNN
 F 2 "Diode_SMD:D_SOD-123" H 7900 5500 50  0001 C CNN
 F 3 "~" H 7900 5500 50  0001 C CNN
@@
 P 9350 5650
 F 0 "D13" V 9350 5800 50  0000 C CNN
-F 1 "MBR0540" V 9700 5650 50  0001 C CNN
+F 1 "F7" V 9700 5650 50  0001 C CNN
 F 2 "Diode_SMD:D_SOD-123" H 9350 5650 50  0001 C CNN
 F 3 "~" H 9350 5650 50  0001 C CNN
