File: kicad/Meteostation_4/Meteostation.sch (KiCad schematic (older format))
At the start: 105 parts, among them J1 TxD, J10 GM+, J11 GM-, J12 SWD, J13 SWC, J2 RxD, J3 BME280_SCL, J4 BME280_SDA, J5 RST, J6 +EXT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

Commit message: новый файл:    Documents/5N10.pdf 	изменено:      kicad/Meteostation_4/Meteostation.kicad_pcb 	изменено:      kicad/Meteostation_4/Meteostation.kicad_pcb-bak 	изменено:      kicad/Meteostation_4/Meteostation.sch 	изменено:      kicad/Meteostation_4/Meteostation.sch-bak 	изменено:      kicad/Meteostation_4/fp-info-cache
Parts:
- removed J8: RxD_AirS8(D8), My-library:SMD-CONN, symbol Connector:Conn_01x01_Female
- removed J9: TxD_AirS8(D9), My-library:SMD-CONN, symbol Connector:Conn_01x01_Female
- C2: footprint Capacitor_SMD:C_1812_4532Metric -> Capacitor_SMD:C_0805_2012Metric
- C21: value 15pF -> 200; footprint Capacitor_SMD:C_0603_1608Metric -> Capacitor_SMD:C_0402_1005Metric
- C22: value 15pF -> 100
- C8: value 480p -> 150nF
- D1: value B82801A1 -> B82801A150
- D10: value MBR0540 -> RS1M; footprint Diode_SMD:D_SOD-123 -> Diode_SMD:D_SMA
- D13: footprint Diode_SMD:D_SOD-123 -> Diode_SMD:D_SMA
- R13: footprint Resistor_SMD:R_1812_4532Metric -> Resistor_SMD:R_1210_3225Metric
- R25: footprint Resistor_SMD:R_0603_1608Metric -> Resistor_SMD:R_0402_1005Metric
- R7: value 10k -> 3.4k
- R8: value 10k -> 1.02k
- Y2: value ECS-250-20-33 -> ECS-250-20-33 25MHz
Connections:
- no-connect marks 35 -> 37
Other:
- moved on the sheet: C1, C17, C18, C2, C20, C22, C25, C26, C6, C8, D10, D15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

Commit message: изменено:      kicad/Meteostation_4/Meteostation-cache.lib 	изменено:      kicad/Meteostation_4/Meteostation-rescue.lib 	изменено:      kicad/Meteostation_4/Meteostation.kicad_pcb 	изменено:      kicad/Meteostation_4/Meteostation.kicad_pcb-bak 	изменено:      kicad/Meteostation_4/Meteostation.sch 	изменено:      kicad/Meteostation_4/Meteostation.sch-bak
Parts:
- added C30, C32: 0.1uF, Capacitor_SMD:C_0603_1608Metric, symbol Device:C
- D1: symbol My_Library:B82801A1 -> Meteostation-rescue:B82801A1-My_Library
- D15: symbol My_Library:SCD41 -> Meteostation-rescue:SCD41-My_Library
Connections:
- wire segments 227 -> 229
Changed lines of the file:
@@
 $EndComp
 $Comp
-L My_Library:B82801A1 D1
+L Meteostation-rescue:B82801A1-My_Library D1
 U 1 1 6364FE98
 P 8000 3100
@@
 NoConn ~ 4850 4850
 $Comp
-L My_Library:SCD41 D15
+L Meteostation-rescue:SCD41-My_Library D15
 U 1 1 640A44F0
 P 10700 4300
@@
 Wire Wire Line
 	8450 7050 9500 7050
+$Comp
+L Device:C C30
+U 1 1 631FC205
+P 11350 4050
+F 0 "C30" H 11300 3750 50  0000 L CNN
+F 1 "0.1uF" H 11250 3650 50  0000 L CNN
+F 2 "Capacitor_SMD:C_0603_1608Metric" H 11388 3900 50  0001 C CNN
+F 3 "~" H 11350 4050 50  0001 C CNN
+	1    11350 4050
+	1    0    0    -1
+$EndComp
+$Comp
+L Device:C C32
+U 1 1 631FD7A8
+P 11550 4050
+F 0 "C32" H 11500 3750 50  0000 L CNN
+F 1 "0.1uF" H 11450 3650 50  0000 L CNN
+F 2 "Capacitor_SMD:C_0603_1608Metric" H 11588 3900 50  0001 C CNN
+F 3 "~" H 11550 4050 50  0001 C CNN
+	1    11550 4050
+	1    0    0    -1
+$EndComp
+Wire Wire Line
+	10900 3900 11350 3900
+Connection ~ 10900 3900
+Connection ~ 11350 3900
+Wire Wire Line
+	11350 3900 11550 3900
+$Comp
+L power:GND #PWR041
+U 1 1 6320F99D
+P 11350 4200
+F 0 "#PWR041" H 11350 3950 50  0001 C CNN
+F 1 "GND" H 11355 4027 50  0001 C CNN
+F 2 "" H 11350 4200 50  0001 C CNN
+F 3 "" H 11350 4200 50  0001 C CNN
+	1    11350 4200
+	1    0    0    -1
+$EndComp
+$Comp
+L power:GND #PWR042
+U 1 1 63210EED
+P 11550 4200
+F 0 "#PWR042" H 11550 3950 50  0001 C CNN
+F 1 "GND" H 11555 4027 50  0001 C CNN
+F 2 "" H 11550 4200 50  0001 C CNN
+F 3 "" H 11550 4200 50  0001 C CNN
+	1    11550 4200
+	1    0    0    -1
+$EndComp
 $EndSCHEMATC

Commit message: изменено:      kicad/Meteostation_4/Meteostation.sch 	изменено:      kicad/Meteostation_4/Meteostation.sch-bak
Parts:
- D13, D8: value MBR0540 -> F7
- D16: value MBR0540 -> SS36
Changed lines of the file:
@@
 P 7900 5500
 F 0 "D8" H 7900 5350 50  0000 C CNN
-F 1 "MBR0540" H 7800 5350 50  0001 C CNN
+F 1 "F7" H 7800 5350 50  0001 C CNN
 F 2 "Diode_SMD:D_SOD-123" H 7900 5500 50  0001 C CNN
 F 3 "~" H 7900 5500 50  0001 C CNN
@@
 P 9350 5650
 F 0 "D13" V 9350 5800 50  0000 C CNN
-F 1 "MBR0540" V 9700 5650 50  0001 C CNN
+F 1 "F7" V 9700 5650 50  0001 C CNN
 F 2 "Diode_SMD:D_SMA" H 9350 5650 50  0001 C CNN
 F 3 "~" H 9350 5650 50  0001 C CNN
@@
 P 10400 5300
 F 0 "D16" H 10450 5000 50  0000 C CNN
-F 1 "MBR0540" H 10450 5100 50  0000 C CNN
+F 1 "SS36" H 10400 5200 50  0000 C CNN
 F 2 "Diode_SMD:D_SOD-128" H 10400 5300 50  0001 C CNN
 F 3 "~" H 10400 5300 50  0001 C CNN
