File: kicad/Meteostation_4/Meteostation.sch (KiCad schematic (older format))
At the start: 105 parts, among them J1 TxD, J10 GM+, J11 GM-, J12 SWD, J13 SWC, J2 RxD, J3 BME280_SCL, J4 BME280_SDA, J5 RST, J6 +EXT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

Commit message: изменено:      kicad/Meteostation_4/Meteostation.kicad_pcb 	изменено:      kicad/Meteostation_4/Meteostation.kicad_pcb-bak 	изменено:      kicad/Meteostation_4/Meteostation.sch 	изменено:      kicad/Meteostation_4/Meteostation.sch-bak 	изменено:      kicad/Meteostation_4/fp-info-cache 	Documents/ATS-1270R.pdf 	Documents/f1-f7.pdf
Parts:
- D13: value F7 -> FR107W F7; footprint Diode_SMD:D_SMA -> Diode_SMD:D_SOD-123F
- D14: value T4932B -> ATS-1270R
- D16: renamed from D; footprint (none) -> Diode_SMD:D_SMA
- D8: value F7 -> FR107W F7; footprint Diode_SMD:D_SOD-123 -> Diode_SMD:D_SOD-123F
- R13: footprint Resistor_SMD:R_1210_3225Metric -> Resistor_SMD:R_1206_3216Metric
Other:
- moved on the sheet: R21, R22
Changed lines of the file:
@@
 P 7900 5500
 F 0 "D8" H 7900 5350 50  0000 C CNN
-F 1 "F7" H 7800 5350 50  0001 C CNN
-F 2 "Diode_SMD:D_SOD-123" H 7900 5500 50  0001 C CNN
+F 1 "FR107W F7" H 7800 5350 50  0001 C CNN
+F 2 "Diode_SMD:D_SOD-123F" H 7900 5500 50  0001 C CNN
 F 3 "~" H 7900 5500 50  0001 C CNN
 	1    7900 5500
@@
 L Device:R R21
 U 1 1 629F9643
-P 7650 5650
-F 0 "R21" H 7850 5700 50  0000 R CNN
-F 1 "43k" H 7850 5600 50  0000 R CNN
-F 2 "Resistor_SMD:R_0603_1608Metric" V 7580 5650 50  0001 C CNN
-F 3 "~" H 7650 5650 50  0001 C CNN
-	1    7650 5650
+P 7700 5650
+F 0 "R21" H 7900 5700 50  0000 R CNN
+F 1 "43k" H 7900 5600 50  0000 R CNN
+F 2 "Resistor_SMD:R_0603_1608Metric" V 7630 5650 50  0001 C CNN
+F 3 "~" H 7700 5650 50  0001 C CNN
+	1    7700 5650
 	1    0    0    -1
 $EndComp
@@
 L Device:R R22
 U 1 1 629F9AAF
-P 7650 6050
+P 7700 6050
 F 0 "R22" H 7850 6250 50  0000 R CNN
-F 1 "10k" H 7850 6150 50  0000 R CNN
-F 2 "Resistor_SMD:R_0603_1608Metric" V 7580 6050 50  0001 C CNN
-F 3 "~" H 7650 6050 50  0001 C CNN
-	1    7650 6050
+F 1 "10k" H 7850 6200 50  0000 R CNN
+F 2 "Resistor_SMD:R_0603_1608Metric" V 7630 6050 50  0001 C CNN
+F 3 "~" H 7700 6050 50  0001 C CNN
+	1    7700 6050
 	1    0    0    -1
 $EndComp
@@
 U 1 1 629FA6A1
 P 8250 5700
-F 0 "C33" V 8150 5350 50  0000 L CNN
-F 1 "480p" V 8250 5350 50  0000 L CNN
+F 0 "C33" V 8150 5450 50  0000 L CNN
+F 1 "480p" V 8200 5450 50  0000 L CNN
 F 2 "Capacitor_SMD:C_0603_1608Metric" H 8288 5550 50  0001 C CNN
 F 3 "~" H 8250 5700 50  0001 C CNN
@@
 P 9350 5650
 F 0 "D13" V 9350 5800 50  0000 C CNN
-F 1 "F7" V 9700 5650 50  0001 C CNN
-F 2 "Diode_SMD:D_SMA" H 9350 5650 50  0001 C CNN
+F 1 "FR107W F7" V 9700 5650 50  0001 C CNN
+F 2 "Diode_SMD:D_SOD-123F" H 9350 5650 50  0001 C CNN
 F 3 "~" H 9350 5650 50  0001 C CNN
 	1    9350 5650
@@
 $EndComp
 $Comp
-L Device:D D
+L Device:D D16
 U 1 1 629FD580
 P 10400 5300
-F 0 "" H 10400 5300 50  0001 C CNN
+F 0 "D16" H 10450 5350 50  0001 C CNN
 F 1 "SS36" H 10400 5200 50  0000 C CNN
-F 2 "" H 10400 5300 50  0001 C CNN
+F 2 "Diode_SMD:D_SMA" H 10400 5300 50  0001 C CNN
 F 3 "~" H 10400 5300 50  0001 C CNN
 	1    10400 5300
@@
 U 1 1 62A36980
 P 8200 5500
-F 0 "R26" V 8350 5650 50  0000 R CNN
+F 0 "R26" V 8450 5450 50  0000 R CNN
 F 1 "20R" V 8350 5450 50  0000 R CNN
 F 2 "Resistor_SMD:R_0603_1608Metric" V 8130 5500 50  0001 C CNN
@@
 Wire Wire Line
 	8400 5400 8400 5500
-Connection ~ 7650 5800
 Wire Wire Line
 	8350 5500 8400 5500
@@
 	7200 7200 7200 7450
 Wire Wire Line
-	7650 5900 7650 5800
-Wire Wire Line
 	9500 6900 9700 6900
 $Comp
@@
 Connection ~ 7500 6200
 Wire Wire Line
-	7500 6200 7650 6200
-Connection ~ 7650 6200
-Wire Wire Line
-	7650 6200 7900 6200
-Wire Wire Line
-	7650 5100 7650 5500
-Wire Wire Line
-	7650 5100 9550 5100
-Wire Wire Line
 	7500 5400 8400 5400
 Connection ~ 7500 5400
 Wire Wire Line
-	7750 5500 7650 5500
-Connection ~ 7650 5500
-Wire Wire Line
-	7650 5800 7900 5800
+	7750 5500 7700 5500
 $Comp
 L Device:C C29
@@
 P 10000 5350
 F 0 "D14" H 10000 5250 50  0000 C CNN
-F 1 "T4932B" H 10000 5700 50  0000 C CNN
+F 1 "ATS-1270R" H 10000 5700 50  0000 C CNN
 F 2 "My-library:DA2257" H 10125 4975 50  0001 C CNN
 F 3 "" H 10125 4975 50  0001 C CNN
@@
 F 0 "R13" H 9300 3200 50  0000 R CNN
 F 1 "5G" H 9250 3100 50  0000 R CNN
-F 2 "Resistor_SMD:R_1210_3225Metric" V 9280 3050 50  0001 C CNN
+F 2 "Resistor_SMD:R_1206_3216Metric" V 9280 3050 50  0001 C CNN
 F 3 "~" H 9350 3050 50  0001 C CNN
 	1    9350 3050
@@
 	10550 5050 10550 5300
 Connection ~ 10550 5300
+Connection ~ 7700 6200
+Wire Wire Line
+	7700 6200 7900 6200
+Connection ~ 7700 5500
+Connection ~ 7700 5800
+Wire Wire Line
+	7700 5800 7900 5800
+Wire Wire Line
+	7500 6200 7700 6200
+Wire Wire Line
+	7700 5900 7700 5800
+Wire Wire Line
+	7700 5500 7700 5100
+Wire Wire Line
+	7700 5100 9550 5100
 $EndSCHEMATC

Commit message: изменено:      kicad/Meteostation_4/Meteostation.sch 	изменено:      kicad/Meteostation_4/Meteostation.sch-bak 	изменено:      stm32cubeide/Meteostation/.mxproject 	изменено:      stm32cubeide/Meteostation/Core/Inc/main.h 	изменено:      stm32cubeide/Meteostation/Core/Inc/stm32f1xx_hal_conf.h 	изменено:      stm32cubeide/Meteostation/Meteostation.ioc 	изменено:      stm32cubeide/Meteostation/Release/Core/Src/BME280.d 	изменено:      stm32cubeide/Meteostation/Release/Core/Src/main.d 	изменено:      stm32cubeide/Meteostation/Release/Core/Src/main.o 	изменено:      stm32cubeide/Meteostation/Release/Core/Src/main.su 	изменено:      stm32cubeide/Meteostation/Release/Core/Src/stm32f1xx_hal_msp.d 	изменено:      stm32cubeide/Meteostation/Release/Core/Src/stm32f1xx_hal_msp.o 	изменено:      stm32cubeide/Meteostation/Release/Core/Src/stm32f1xx_hal_msp.su 	изменено:      stm32cubeide/Meteostation/Release/Core/Src/stm32f1xx_it.d 	изменено:      stm32cubeide/Meteostation/Release/Core/Src/stm32f1xx_it.o 	изменено:      stm32cubeide/Meteostation/Release/Core/Src/system_stm32f1xx.d 	изменено:      stm32cubeide/Meteostation/Release/Drivers/STM32F1xx_HAL_Driver/Src/stm32f1xx_hal.d 	изменено:      stm32cubeide/Meteostation/Release/Drivers/STM32F1xx_HAL_Driver/Src/stm32f1xx_hal_cortex.d 	изменено:      stm32cubeide/Meteostation/Release/Drivers/STM32F1xx_HAL_Driver/Src/stm32f1xx_hal_dma.d 	изменено:      stm32cubeide/Meteostation/Release/Drivers/STM32F1xx_HAL_Driver/Src/stm32f1xx_hal_exti.d 	изменено:      stm32cubeide/Meteostation/Release/Drivers/STM32F1xx_HAL_Driver/Src/stm32f1xx_hal_flash.d 	изменено:      stm32cubeide/Meteostation/Release/Drivers/STM32F1xx_HAL_Driver/Src/stm32f1xx_hal_flash_ex.d 	изменено:      stm32cubeide/Meteostation/Release/Drivers/STM32F1xx_HAL_Driver/Src/stm32f1xx_hal_gpio.d 	изменено:      stm32cubeide/Meteostation/Release/Drivers/STM32F1xx_HAL_Driver/Src/stm32f1xx_hal_gpio_ex.d 	изменено:      stm32cubeide/Meteostation/Release/Drivers/STM32F1xx_HAL_Driver/S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
Parts:
- D10: value RS1M -> SS510
Changed lines of the file:
@@
 P 8900 4700
 F 0 "D10" V 8900 4550 50  0000 C CNN
-F 1 "RS1M" H 8800 4550 50  0001 C CNN
+F 1 "SS510" H 8800 4550 50  0001 C CNN
 F 2 "Diode_SMD:D_SMA" H 8900 4700 50  0001 C CNN
 F 3 "~" H 8900 4700 50  0001 C CNN

Commit message: изменено:      kicad/Meteostation_4/Meteostation.kicad_pcb 	изменено:      kicad/Meteostation_4/Meteostation.kicad_pcb-bak 	изменено:      kicad/Meteostation_4/Meteostation.sch 	изменено:      kicad/Meteostation_4/Meteostation.sch-bak 	изменено:      kicad/Meteostation_4/fp-info-cache
Parts:
- D10: value SS510 -> SS56
- R5: value 10 -> 47
Changed lines of the file:
@@
 P 8900 4700
 F 0 "D10" V 8900 4550 50  0000 C CNN
-F 1 "SS510" H 8800 4550 50  0001 C CNN
+F 1 "SS56" H 8800 4550 50  0001 C CNN
 F 2 "Diode_SMD:D_SMA" H 8900 4700 50  0001 C CNN
 F 3 "~" H 8900 4700 50  0001 C CNN
@@
 P 7350 2800
 F 0 "R5" V 7150 2850 50  0000 R CNN
-F 1 "10" V 7250 2850 50  0000 R CNN
+F 1 "47" V 7250 2850 50  0000 R CNN
 F 2 "Resistor_SMD:R_0603_1608Metric" V 7280 2800 50  0001 C CNN
 F 3 "~" H 7350 2800 50  0001 C CNN

Commit message: изменено:      kicad/Meteostation_4/Meteostation.kicad_pcb 	изменено:      kicad/Meteostation_4/Meteostation.kicad_pcb-bak 	изменено:      kicad/Meteostation_4/Meteostation.sch 	изменено:      kicad/Meteostation_4/Meteostation.sch-bak
Parts:
- removed J5: RST, My-library:SMD-CONN, symbol Connector:Conn_01x01_Female
- added R6: 100k, Resistor_SMD:R_0603_1608Metric, symbol Device:R
Connections:
- net GND: now also R6.2
- net PWR: now also R6.1
Changed lines of the file:
@@
 	4500 3350 4850 3350
-$Comp
-L Connector:Conn_01x01_Female J5
-U 1 1 632E013C
-P 4500 3150
-F 0 "J5" V 4650 3150 50  0001 C CNN
-F 1 "RST" V 4400 3250 50  0000 L CNN
-F 2 "My-library:SMD-CONN" H 4500 3150 50  0001 C CNN
-F 3 "~" H 4500 3150 50  0001 C CNN
-	1    4500 3150
-	0    -1   -1   0
-$EndComp
-Connection ~ 4500 3350
 $Comp
 L Regulator_Switching:LMR14206 U2
@@
 	7800 3650 7800 3700
 Connection ~ 7800 3650
-Text GLabel 7500 3400 0    50   Input ~ 0
+Text GLabel 7400 3400 0    50   Input ~ 0
 PWR
 $Comp
@@
 Wire Wire Line
 	7700 5100 9550 5100
+$Comp
+L Device:R R6
+U 1 1 634FB19F
+P 7500 3550
+F 0 "R6" H 7250 3550 50  0000 R CNN
+F 1 "100k" H 7300 3450 50  0000 R CNN
+F 2 "Resistor_SMD:R_0603_1608Metric" V 7430 3550 50  0001 C CNN
+F 3 "~" H 7500 3550 50  0001 C CNN
+	1    7500 3550
+	1    0    0    -1
+$EndComp
+$Comp
+L power:GND #PWR043
+U 1 1 63505702
+P 7500 3700
+F 0 "#PWR043" H 7500 3450 50  0001 C CNN
+F 1 "GND" H 7505 3527 50  0001 C CNN
+F 2 "" H 7500 3700 50  0001 C CNN
+F 3 "" H 7500 3700 50  0001 C CNN
+	1    7500 3700
+	1    0    0    -1
+$EndComp
+Wire Wire Line
+	7400 3400 7500 3400
+Connection ~ 7500 3400
 $EndSCHEMATC
