File: kicad/Meteostation_4/Meteostation.sch (KiCad schematic (older format))
At the start: 112 parts, among them J1 TxD, J10 GM+, J11 GM-, J12 SWD, J13 SWC, J14 DISP_CS, J15 OLED_SCL, J16 OLED_SDA, J2 RxD, J3 BME280_SCL, J4 BME280_SDA, J5 miso, J6 +EXT, J7 -EXT, J8 mosi, J9 sclk, Q1 5N10, Q2 IRLML6346, Q3 Q_NPN_BEC, T1 HY931147C, U1 STM32F103C8Tx, U2 LMR14206, U3 AD8541, Y2 ECS-250-20-33 25MHz

Commit message: изменено:      Arduino/meteomonitor/meteomonitor.ino 	изменено:      FreeCAD/GM_case_top.FCStd 	изменено:      kicad/Meteostation_4/Meteostation-cache.lib 	изменено:      kicad/Meteostation_4/Meteostation-rescue.lib 	изменено:      kicad/Meteostation_4/Meteostation.kicad_pcb 	изменено:      kicad/Meteostation_4/Meteostation.kicad_pcb-bak 	изменено:      kicad/Meteostation_4/Meteostation.sch 	изменено:      kicad/Meteostation_4/Meteostation.sch-bak 	изменено:      kicad/Meteostation_4/fp-info-cache 	изменено:      stm32cubeide/Meteostation/.cproject 	изменено:      stm32cubeide/Meteostation/.mxproject 	изменено:      stm32cubeide/Meteostation/.settings/language.settings.xml 	изменено:      stm32cubeide/Meteostation/Core/Inc/main.h 	изменено:      stm32cubeide/Meteostation/Core/Inc/stm32f1xx_it.h 	изменено:      stm32cubeide/Meteostation/Core/Src/BME280.c 	изменено:      stm32cubeide/Meteostation/Core/Src/main.c 	изменено:      stm32cubeide/Meteostation/Core/Src/stm32f1xx_hal_msp.c 	изменено:      stm32cubeide/Meteostation/Core/Src/stm32f1xx_it.c 	изменено:      stm32cubeide/Meteostation/Meteostation.ioc 	изменено:      stm32cubeide/Meteostation/Meteostation.launch 	изменено:      stm32cubeide/Meteostation/Release/Core/Src/BME280.d 	изменено:      stm32cubeide/Meteostation/Release/Core/Src/BME280.o 	изменено:      stm32cubeide/Meteostation/Release/Core/Src/main.d 	изменено:      stm32cubeide/Meteostation/Release/Core/Src/main.o 	изменено:      stm32cubeide/Meteostation/Release/Core/Src/main.su 	изменено:      stm32cubeide/Meteostation/Release/Core/Src/stm32f1xx_hal_msp.d 	изменено:      stm32cubeide/Meteostation/Release/Core/Src/stm32f1xx_hal_msp.o 	изменено:      stm32cubeide/Meteostation/Release/Core/Src/stm32f1xx_hal_msp.su 	изменено:      stm32cubeide/Meteostation/Release/Core/Src/stm32f1xx_it.d 	изменено:      stm32cubeide/Meteostation/Release/Core/Src/stm32f1xx_it.o 	изменено:      stm32cubeide/Meteostation/Release/Core/Src/stm32f1xx_it.su 	изменено:      stm32c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
Parts:
- removed J5: miso, My-library:ConnMini, symbol Connector:Conn_01x01_Female
- added J17: ST7735S_DC, My-library:mini_conn, symbol Connector:Conn_01x01_Female
- added J18: ST7735S_RESET, My-library:mini_conn, symbol Connector:Conn_01x01_Female
- D15: symbol My_Library:SCD41 -> Meteostation-rescue:SCD41-My_Library
- J14: value DISP_CS -> ST7735S_CS; footprint My-library:ConnMini -> My-library:mini_conn
- R4: value 1k -> 4.7k
Connections:
- net at U1.22 (PB11): now also J18.1 (Pin_1)
- net at U1.31 (PA10): now also J17.1 (Pin_1)
- no-connect marks 36 -> 34
Changed lines of the file:
@@
 U 1 1 61E82A7E
 P 6500 5650
-F 0 "R4" V 6300 5700 50  0000 R CNN
-F 1 "1k" V 6400 5700 50  0000 R CNN
+F 0 "R4" V 6400 6000 50  0000 R CNN
+F 1 "4.7k" V 6500 6000 50  0000 R CNN
 F 2 "Resistor_SMD:R_0402_1005Metric" V 6430 5650 50  0001 C CNN
 F 3 "~" H 6500 5650 50  0001 C CNN
@@
 NoConn ~ 4850 4950
 NoConn ~ 6150 5150
-NoConn ~ 6150 5450
 NoConn ~ 6150 5550
 NoConn ~ 4850 5450
-NoConn ~ 4850 5550
 $Comp
 L Device:C C22
@@
 P 6350 5350
 F 0 "J14" H 6600 5350 50  0001 C CNN
-F 1 "DISP_CS" H 6350 5350 50  0000 L CNN
-F 2 "My-library:ConnMini" H 6350 5350 50  0001 C CNN
+F 1 "ST7735S_CS" H 6350 5350 50  0000 L CNN
+F 2 "My-library:mini_conn" H 6350 5350 50  0001 C CNN
 F 3 "~" H 6350 5350 50  0001 C CNN
 	1    6350 5350
-	1    0    0    -1
-$EndComp
-$Comp
-L Connector:Conn_01x01_Female J5
-U 1 1 638107F7
-P 5050 6350
-F 0 "J5" H 5300 6350 50  0001 C CNN
-F 1 "miso" H 5050 6350 50  0001 L CNN
-F 2 "My-library:ConnMini" H 5050 6350 50  0001 C CNN
-F 3 "~" H 5050 6350 50  0001 C CNN
-	1    5050 6350
 	1    0    0    -1
 $EndComp
@@
 	1    0    0    -1
 $EndComp
-Text GLabel 4850 6350 0    50   Input ~ 0
-MISO
 Text GLabel 4850 6450 0    50   Input ~ 0
 MOSI
@@
 Connection ~ 7500 4100
 $Comp
-L My_Library:SCD41 D15
+L Meteostation-rescue:SCD41-My_Library D15
 U 1 1 63BEA614
 P 10250 4300
@@
 	4350 5600 4250 5600
 Connection ~ 4350 5500
+$Comp
+L Connector:Conn_01x01_Female J17
+U 1 1 647DE59A
+P 6350 5450
+F 0 "J17" H 6600 5450 50  0001 C CNN
+F 1 "ST7735S_DC" H 6350 5450 50  0000 L CNN
+F 2 "My-library:mini_conn" H 6350 5450 50  0001 C CNN
+F 3 "~" H 6350 5450 50  0001 C CNN
+	1    6350 5450
+	1    0    0    -1
+$EndComp
+$Comp
+L Connector:Conn_01x01_Female J18
+U 1 1 647E2272
+P 4650 5550
+F 0 "J18" H 4900 5550 50  0001 C CNN
+F 1 "ST7735S_RESET" H 4700 5700 50  0000 L CNN
+F 2 "My-library:mini_conn" H 4650 5550 50  0001 C CNN
+F 3 "~" H 4650 5550 50  0001 C CNN
+	1    4650 5550
+	-1   0    0    1
+$EndComp
+Text Label 4850 6450 0    50   ~ 0
+ST7735_SDA
+Text Label 4850 6550 0    50   ~ 0
+ST7735_SCK
 $EndSCHEMATC

Commit message: изменено:      kicad/Meteostation_4/Meteostation.kicad_pcb 	изменено:      kicad/Meteostation_4/Meteostation.kicad_pcb-bak 	изменено:      kicad/Meteostation_4/Meteostation.sch 	изменено:      kicad/Meteostation_4/Meteostation.sch-bak 	изменено:      kicad/Meteostation_4/gerber/Border.gbr 	изменено:      kicad/Meteostation_4/gerber/Bottom.gbr 	изменено:      kicad/Meteostation_4/gerber/MaskBottom.gbr 	изменено:      kicad/Meteostation_4/gerber/MaskTop.gbr 	изменено:      kicad/Meteostation_4/gerber/Meteostation-job.gbrjob 	изменено:      kicad/Meteostation_4/gerber/Meteostation.zip 	изменено:      kicad/Meteostation_4/gerber/NCData.drl 	изменено:      kicad/Meteostation_4/gerber/Top.gbr
Parts:
- removed D10: SS56, VS10MQ060-M3/5, Diode_SMD:D_SMA, symbol Device:D
- added J5: +EXT, My-library:ConnMini, symbol Connector:Conn_01x01_Female
- C19: value 22uF/63v -> 100uF/63v; footprint Capacitor_SMD:CP_Elec_6.3x7.7 -> My-library:CAP_horizontal
- C22: footprint Capacitor_SMD:C_0603_1608Metric -> Capacitor_SMD:C_0402_1005Metric
- R13: value 5G -> HVC1206Z5007KET
- R16: footprint Resistor_SMD:R_0603_1608Metric -> Resistor_SMD:R_0402_1005Metric
- U2: value LMR14206 -> LMR50410XDBVR
Connections:
- net +3.3VDAC: now also J5.1 (Pin_1)
Changed lines of the file:
@@
 U 1 1 629FA6A1
 P 8250 5700
-F 0 "C33" V 8200 5400 50  0000 L CNN
-F 1 "480p" V 8300 5350 50  0000 L CNN
+F 0 "C33" V 8150 5400 50  0000 L CNN
+F 1 "480p" V 8250 5350 50  0000 L CNN
 F 2 "Capacitor_SMD:C_0603_1608Metric" H 8288 5550 50  0001 C CNN
 F 3 "~" H 8250 5700 50  0001 C CNN
@@
 P 7200 6050
 F 0 "C19" H 7000 6200 50  0000 L CNN
-F 1 "22uF/63v" H 7000 5850 50  0000 L CNN
-F 2 "Capacitor_SMD:CP_Elec_6.3x7.7" H 7238 5900 50  0001 C CNN
+F 1 "100uF/63v" H 7000 5850 50  0000 L CNN
+F 2 "My-library:CAP_horizontal" H 7238 5900 50  0001 C CNN
 F 3 "~" H 7200 6050 50  0001 C CNN
 	1    7200 6050
@@
 P 8000 4300
 F 0 "U2" H 8000 4550 50  0000 C CNN
-F 1 "LMR14206" H 8000 4400 50  0000 C CNN
+F 1 "LMR50410XDBVR" H 8000 4400 50  0000 C CNN
 F 2 "Package_TO_SOT_SMD:SOT-23-6" H 8000 3800 50  0001 C CIN
 F 3 "http://www.ti.com/lit/ds/symlink/lmr14206.pdf" H 7600 4750 50  0001 C CNN
@@
 	1    9100 4700
 	1    0    0    -1
-$EndComp
-$Comp
-L Device:D D10
-U 1 1 63393350
-P 8800 4700
-F 0 "D10" V 8800 4550 50  0000 C CNN
-F 1 "SS56, VS10MQ060-M3/5" H 8700 4550 50  0001 C CNN
-F 2 "Diode_SMD:D_SMA" H 8800 4700 50  0001 C CNN
-F 3 "~" H 8800 4700 50  0001 C CNN
-	1    8800 4700
-	0    1    1    0
 $EndComp
 $Comp
@@
 Connection ~ 8000 4900
 Wire Wire Line
-	8800 4300 8800 4550
-Connection ~ 8800 4300
-Wire Wire Line
 	9100 4900 9100 4850
-Wire Wire Line
-	8000 4900 8800 4900
-Wire Wire Line
-	8800 4850 8800 4900
-Connection ~ 8800 4900
-Wire Wire Line
-	8800 4900 9100 4900
 Wire Wire Line
 	9100 4550 9100 4500
@@
 L power:+3.3VDAC #PWR01
 U 1 1 635A6E73
-P 4600 7000
-F 0 "#PWR01" H 4750 6950 50  0001 C CNN
-F 1 "+3.3VDAC" H 4650 7100 50  0000 L CNN
-F 2 "" H 4600 7000 50  0001 C CNN
-F 3 "" H 4600 7000 50  0001 C CNN
-	1    4600 7000
+P 4600 6850
+F 0 "#PWR01" H 4750 6800 50  0001 C CNN
+F 1 "+3.3VDAC" H 4650 6950 50  0000 L CNN
+F 2 "" H 4600 6850 50  0001 C CNN
+F 3 "" H 4600 6850 50  0001 C CNN
+	1    4600 6850
 	1    0    0    -1
 $EndComp
@@
 P 9050 2950
 F 0 "R13" H 9000 3100 50  0000 R CNN
-F 1 "5G" H 8950 3000 50  0000 R CNN
+F 1 "HVC1206Z5007KET" H 9800 3100 50  0000 R CNN
 F 2 "Resistor_SMD:R_1206_3216Metric" V 8980 2950 50  0001 C CNN
 F 3 "~" H 9050 2950 50  0001 C CNN
@@
 F 0 "C22" H 9100 3150 50  0000 L CNN
 F 1 "100" H 9100 3250 50  0000 L CNN
-F 2 "Capacitor_SMD:C_0603_1608Metric" H 9088 3200 50  0001 C CNN
+F 2 "Capacitor_SMD:C_0402_1005Metric" H 9088 3200 50  0001 C CNN
 F 3 "~" H 9050 3350 50  0001 C CNN
 	1    9050 3350
@@
 F 0 "R16" H 9350 3750 50  0000 R CNN
 F 1 "10M" H 9350 3650 50  0000 R CNN
-F 2 "Resistor_SMD:R_0603_1608Metric" V 9180 3350 50  0001 C CNN
+F 2 "Resistor_SMD:R_0402_1005Metric" V 9180 3350 50  0001 C CNN
 F 3 "~" H 9250 3350 50  0001 C CNN
 	1    9250 3350
@@
 Text Label 4850 6550 0    50   ~ 0
 ST7735_SCK
+Wire Wire Line
+	8000 4900 9100 4900
+$Comp
+L Connector:Conn_01x01_Female J5
+U 1 1 64897F7B
+P 4400 6900
+F 0 "J5" H 3900 6900 50  0001 C CNN
+F 1 "+EXT" H 4400 6900 50  0000 L CNN
+F 2 "My-library:ConnMini" H 4400 6900 50  0001 C CNN
+F 3 "~" H 4400 6900 50  0001 C CNN
+	1    4400 6900
+	-1   0    0    1
+$EndComp
+Wire Wire Line
+	4600 7000 4600 6900
+Connection ~ 4600 6900
+Wire Wire Line
+	4600 6900 4600 6850
 $EndSCHEMATC
