File: kicad/Meteostation_4/Meteostation.kicad_pcb (KiCad board)
At the start: 2 copper layers, 44 x 44 mm, 105 parts, among them J1 TxD, J10 GM+, J11 GM-, J12 SWD, J13 SWC, J2 RxD, J3 BME280_SCL, J4 BME280_SDA, J6 +EXT, J7 -EXT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

Commit message: изменено:      kicad/Meteostation_4/Meteostation.kicad_pcb 	изменено:      kicad/Meteostation_4/Meteostation.kicad_pcb-bak 	изменено:      kicad/Meteostation_4/Meteostation.pro 	изменено:      kicad/Meteostation_4/Meteostation.sch 	изменено:      kicad/Meteostation_4/Meteostation.sch-bak 	изменено:      kicad/Meteostation_4/fp-info-cache
Parts:
- added R29: 0, Resistor_SMD:R_1206_3216Metric, F.Cu at (43.2, 95.2)
- C1, C30, C8, D10, L2, R7, R8, U2: moved to B.Cu
- C17, C3, C6: footprint Capacitor_SMD:C_1812_4532Metric -> Capacitor_SMD:C_1206_3216Metric
- C32, D15: moved to F.Cu
- R5: footprint Resistor_SMD:R_0603_1608Metric -> Resistor_SMD:R_1206_3216Metric
- moved R15 15.1 mm to (45.2, 68.3)
- moved D5 14.4 mm to (45.2, 71.3)
- moved C32 12.6 mm to (51.6, 81.3), turned to 90 degrees
- moved J6 12.1 mm to (46.6, 92.2)
- moved C30 11.2 mm to (35.3, 82.5), turned to 270 degrees
- moved C18 10.6 mm to (37.2, 84.1)
- moved R8 9.29 mm to (36.7, 82.5), turned to 270 degrees
- moved R7 6.53 mm to (39.3, 82.2), turned to 180 degrees
- moved L2 6.39 mm to (45.6, 84.8), turned to 90 degrees
- moved D15 5.51 mm to (45.6, 83.4), turned to 270 degrees
- moved C1 4.25 mm to (39.1, 84.0), turned to 180 degrees
- moved C3 3.29 mm to (41.8, 93.5)
- moved C2 3.00 mm to (37.1, 93.6)
- moved Q2 3.00 mm to (37.2, 96.3)
- moved R6 3.00 mm to (39.5, 94.5)
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Connections:
- Q2 pad 1: PWR -> Net-(Q2-Pad1)
- R6 pad 1: PWR -> Net-(Q2-Pad1)
Routing:
- net GND: track 189.9 -> 167.0 mm, vias 12 -> 10
- net +3.3VDAC: track 115.0 -> 110.0 mm
- net SDA: track 24.8 -> 20.9 mm, vias 1 -> 0
- net Net-(C2-Pad1): track 3.11 -> 6.89 mm
- net 12-16: track 17.0 -> 13.3 mm, vias 1 -> 2
- net Net-(Q2-Pad1): track 0.00 -> 3.57 mm
- net PWR: track 7.47 -> 3.98 mm
- net Net-(C8-Pad2): track 8.72 -> 11.7 mm
- net SCL: track 24.4 -> 21.6 mm, vias 1 -> 2
- net Net-(J2-Pad1): track 4.57 -> 1.92 mm
- net Net-(C17-Pad1): track 6.74 -> 5.42 mm
- net Net-(C19-Pad1): track 93.8 -> 92.9 mm
- net Net-(J13-Pad1): track 2.42 -> 1.82 mm
- net Net-(R7-Pad2): track 5.64 -> 6.20 mm
- net Net-(C3-Pad2): track 4.57 -> 4.03 mm
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Other:
- net class Default: via_dia 0.8 -> 1
